Commit message: 完成了雷达部署

File: src/sensor_fusion_robot/urdf/robot.urdf.xacro (robot description, xacro)
@@ -10,4 +10,7 @@
   <material name="white">
     <color rgba="1 1 1 1"/>
+  </material>
+  <material name="red">
+    <color rgba="0.8 0 0 1"/>
   </material>
   <!-- 底盘尺寸参数 -->
@@ -205,6 +208,29 @@
     <parent link="sensor_platform_link"/>
     <child link="lidar_link"/>
-    <origin xyz="0 0 0.06" rpy="0 0 0"/>
-  </joint>
+    <origin xyz="0 0 0.1" rpy="0 0 0"/>
+  </joint>
+  <!-- IMU模型 -->
+  <link name="imu_link">
+    <visual>
+      <geometry>
+        <box size="0.03 0.03 0.01"/>
+      </geometry>
+      <material name="red"/>
+    </visual>
+    <collision>
+      <geometry>
+        <box size="0.03 0.03 0.01"/>
+      </geometry>
+    </collision>
+    <xacro:box_inertia mass="0.01" x="0.03" y="0.03" z="0.01"/>
+  </link>
+  <joint name="imu_joint" type="fixed">
+    <parent link="sensor_platform_link"/>
+    <child link="imu_link"/>
+    <origin xyz="0.05 0 0.015" rpy="0 0 0"/>
+  </joint>
+  <gazebo reference="imu_link">
+    <material>Gazebo/Red</material>
+  </gazebo>
   <!-- Gazebo配置 -->
   <gazebo reference="base_link">
@@ -287,13 +313,19 @@
       <scan>
         <horizontal>
-          <samples>360</samples>
+          <samples>640</samples>
           <resolution>1</resolution>
-          <min_angle>-3.14159</min_angle>
-          <max_angle>3.14159</max_angle>
+          <min_angle>-1.396263</min_angle>
+          <max_angle>1.396263</max_angle>
         </horizontal>
+        <vertical>
+          <samples>32</samples>
+          <resolution>1</resolution>
+          <min_angle>-0.261799</min_angle>
+          <max_angle>0.261799</max_angle>
+        </vertical>
       </scan>
       <range>
-        <min>0.12</min>
-        <max>6.0</max>
+        <min>0.08</min>
+        <max>10.0</max>
         <resolution>0.01</resolution>
       </range>
@@ -310,6 +342,9 @@
       <topic>gazebo_ros_lidar/out</topic>
       <frame_name>lidar_link</frame_name>
+      <output_type>PointCloud2</output_type>
     </plugin>
   </sensor>
 </gazebo>
+  <! -- Todo: 修改雷达，使用https://github.com/stm32f303ret6/livox_laser_simulation_RO2的模型 -->
+  <!-- IMU Gazebo插件 -->
 </robot>

Commit message: 部署了三维Libar mid360，完成其测试

File: src/sensor_fusion_robot/urdf/robot.urdf.xacro (robot description, xacro)
@@ -1,4 +1,5 @@
 <?xml version="1.0"?>
 <robot xmlns:xacro="http://www.ros.org/wiki/xacro" name="sensor_fusion_robot">
+<xacro:include filename="$(find ros2_livox_simulation)/urdf/mid360.xacro" />
   <!-- 材质定义 -->
   <material name="blue">
@@ -26,5 +27,5 @@
   <xacro:property name="wheel_offset_z" value="-0.05"/>
   <!-- 惯性宏定义 -->
-  <xacro:macro name="box_inertia" params="mass x y z">
+  <xacro:macro name="robot_box_inertia" params="mass x y z">
     <inertial>
       <origin xyz="0 0 0" rpy="0 0 0"/>
@@ -90,5 +91,5 @@
       </geometry>
     </collision>
-    <xacro:box_inertia mass="${chassis_mass}" x="${chassis_length}" y="${chassis_width}" z="${chassis_height}"/>
+    <xacro:robot_box_inertia mass="${chassis_mass}" x="${chassis_length}" y="${chassis_width}" z="${chassis_height}"/>
   </link>
   <!-- 添加轮子 -->
@@ -153,5 +154,5 @@
       </geometry>
     </collision>
-    <xacro:box_inertia mass="0.5" x="${chassis_length/2}" y="${chassis_width/2}" z="0.02"/>
+    <xacro:robot_box_inertia mass="0.5" x="${chassis_length/2}" y="${chassis_width/2}" z="0.02"/>
   </link>
   <joint name="sensor_platform_joint" type="fixed">
@@ -175,5 +176,5 @@
       </geometry>
     </collision>
-    <xacro:box_inertia mass="0.1" x="0.05" y="0.05" z="0.05"/>
+    <xacro:robot_box_inertia mass="0.1" x="0.05" y="0.05" z="0.05"/>
   </link>
   <joint name="camera_joint" type="fixed">
@@ -182,32 +183,4 @@
     <origin xyz="0 0 0.05" rpy="0 0 0"/>
   </joint>
-  <!-- Lidar模型 -->
-  <link name="lidar_link">
-    <visual>
-      <origin xyz="0 0 0" rpy="0 0 0"/>
-      <geometry>
-        <cylinder radius="0.04" length="0.08"/>
-      </geometry>
-      <material name="black"/>
-    </visual>
-    <collision>
-      <origin xyz="0 0 0" rpy="0 0 0"/>
-      <geometry>
-        <cylinder radius="0.04" length="0.08"/>
-      </geometry>
-    </collision>
-    <inertial>
-      <origin xyz="0 0 0" rpy="0 0 0"/>
-      <mass value="0.2"/>
-      <inertia ixx="0.0001" ixy="0.0" ixz="0.0"
-               iyy="0.0001" iyz="0.0"
-               izz="0.0002"/>
-    </inertial>
-  </link>
-    <joint name="lidar_joint" type="fixed">
-    <parent link="sensor_platform_link"/>
-    <child link="lidar_link"/>
-    <origin xyz="0 0 0.1" rpy="0 0 0"/>
-  </joint>
   <!-- IMU模型 -->
   <link name="imu_link">
@@ -223,5 +196,5 @@
       </geometry>
     </collision>
-    <xacro:box_inertia mass="0.01" x="0.03" y="0.03" z="0.01"/>
+    <xacro:robot_box_inertia mass="0.01" x="0.03" y="0.03" z="0.01"/>
   </link>
   <joint name="imu_joint" type="fixed">
@@ -233,4 +206,8 @@
     <material>Gazebo/Red</material>
   </gazebo>
+  <!-- Mid360 雷达 -->
+  <xacro:mid360 name="mid360" parent="sensor_platform_link" topic="mid360">
+    <origin xyz="0 0 0.1" rpy="0 0 0"/>
+  </xacro:mid360>
   <!-- Gazebo配置 -->
   <gazebo reference="base_link">
@@ -331,5 +308,5 @@
       </range>
       <noise>
-        <type>gaussian</type>
+        <type>gaussian</type>xacro:mid70
         <mean>0.0</mean>
         <stddev>0.01</stddev>
@@ -346,5 +323,3 @@
   </sensor>
 </gazebo>
-  <! -- Todo: 修改雷达，使用https://github.com/stm32f303ret6/livox_laser_simulation_RO2的模型 -->
-  <!-- IMU Gazebo插件 -->
 </robot>
